File: hardware/MCU.sch (KiCad schematic (older format))
At the start: 5 parts

Commit message: HC49-U
Parts:
- Y?: footprint (none) -> Crystal:Crystal_HC49-U_Vertical
Changed lines of the file:
@@
 F 0 "Y?" H 4800 2768 50  0000 C CNN
 F 1 "16MHz" H 4800 2677 50  0000 C CNN
-F 2 "" H 4800 2500 50  0001 C CNN
+F 2 "Crystal:Crystal_HC49-U_Vertical" H 4800 2500 50  0001 C CNN
 F 3 "~" H 4800 2500 50  0001 C CNN
 	1    4800 2500

Commit message: Updated PCB
Parts:
- C1: renamed from C?; value C -> 1u; footprint (none) -> Capacitor_THT:C_Rect_L7.2mm_W4.5mm_P5.00mm_FKS2_FKP2_MKS2_MKP2
- C2, C3: renamed from C?; footprint (none) -> Capacitor_THT:C_Disc_D3.8mm_W2.6mm_P2.50mm
- gave numbers to parts that had none: 2
Changed lines of the file:
@@
 $EndDescr
 $Comp
-L MCU_Microchip_ATmega:ATmega328P-PU U?
+L MCU_Microchip_ATmega:ATmega328P-PU U1
 U 1 1 5EB47D68
 P 2850 2750
-F 0 "U?" H 2206 2796 50  0000 R CNN
+F 0 "U1" H 2206 2796 50  0000 R CNN
 F 1 "ATmega328P-PU" H 2206 2705 50  0000 R CNN
 F 2 "Package_DIP:DIP-28_W7.62mm" H 2850 2750 50  0001 C CIN
@@
 $EndComp
 $Comp
-L Device:Crystal Y?
+L Device:Crystal Y1
 U 1 1 5EB530DB
 P 4800 2500
-F 0 "Y?" H 4800 2768 50  0000 C CNN
+F 0 "Y1" H 4800 2768 50  0000 C CNN
 F 1 "16MHz" H 4800 2677 50  0000 C CNN
 F 2 "Crystal:Crystal_HC49-U_Vertical" H 4800 2500 50  0001 C CNN
@@
 $EndComp
 $Comp
-L Device:C C?
+L Device:C C2
 U 1 1 5EB538EA
 P 4550 2750
-F 0 "C?" H 4665 2796 50  0000 L CNN
+F 0 "C2" H 4665 2796 50  0000 L CNN
 F 1 "22p" H 4665 2705 50  0000 L CNN
-F 2 "" H 4588 2600 50  0001 C CNN
+F 2 "Capacitor_THT:C_Disc_D3.8mm_W2.6mm_P2.50mm" H 4588 2600 50  0001 C CNN
 F 3 "~" H 4550 2750 50  0001 C CNN
 	1    4550 2750
@@
 $EndComp
 $Comp
-L Device:C C?
+L Device:C C3
 U 1 1 5EB53C11
 P 5050 2750
-F 0 "C?" H 5165 2796 50  0000 L CNN
+F 0 "C3" H 5165 2796 50  0000 L CNN
 F 1 "22p" H 5165 2705 50  0000 L CNN
-F 2 "" H 5088 2600 50  0001 C CNN
+F 2 "Capacitor_THT:C_Disc_D3.8mm_W2.6mm_P2.50mm" H 5088 2600 50  0001 C CNN
 F 3 "~" H 5050 2750 50  0001 C CNN
 	1    5050 2750
@@
 $EndComp
 $Comp
-L power:GND #PWR?
+L power:GND #PWR0101
 U 1 1 5EB5525A
 P 2850 4350
-F 0 "#PWR?" H 2850 4100 50  0001 C CNN
+F 0 "#PWR0101" H 2850 4100 50  0001 C CNN
 F 1 "GND" H 2855 4177 50  0000 C CNN
 F 2 "" H 2850 4350 50  0001 C CNN
@@
 	2850 4250 2850 4350
 $Comp
-L power:GND #PWR?
+L power:GND #PWR0102
 U 1 1 5EB55CD3
 P 4800 3100
-F 0 "#PWR?" H 4800 2850 50  0001 C CNN
+F 0 "#PWR0102" H 4800 2850 50  0001 C CNN
 F 1 "GND" H 4805 2927 50  0000 C CNN
 F 2 "" H 4800 3100 50  0001 C CNN
@@
 Connection ~ 4550 2500
 $Comp
-L Device:C C?
+L Device:C C1
 U 1 1 5EB5C7A4
 P 1550 1400
-F 0 "C?" H 1665 1446 50  0000 L CNN
-F 1 "C" H 1665 1355 50  0000 L CNN
-F 2 "" H 1588 1250 50  0001 C CNN
+F 0 "C1" H 1665 1446 50  0000 L CNN
+F 1 "1u" H 1665 1355 50  0000 L CNN
+F 2 "Capacitor_THT:C_Rect_L7.2mm_W4.5mm_P5.00mm_FKS2_FKP2_MKS2_MKP2" H 1588 1250 50  0001 C CNN
 F 3 "~" H 1550 1400 50  0001 C CNN
 	1    1550 1400
@@
 $EndComp
 $Comp
-L power:+5V #PWR?
+L power:+5V #PWR0103
 U 1 1 5EB5DB30
 P 1550 1050
-F 0 "#PWR?" H 1550 900 50  0001 C CNN
+F 0 "#PWR0103" H 1550 900 50  0001 C CNN
 F 1 "+5V" H 1565 1223 50  0000 C CNN
 F 2 "" H 1550 1050 50  0001 C CNN
@@
 $EndComp
 $Comp
-L power:GND #PWR?
+L power:GND #PWR0104
 U 1 1 5EB5EFDF
 P 1550 1650
-F 0 "#PWR?" H 1550 1400 50  0001 C CNN
+F 0 "#PWR0104" H 1550 1400 50  0001 C CNN
 F 1 "GND" H 1555 1477 50  0000 C CNN
 F 2 "" H 1550 1650 50  0001 C CNN

Commit message: Added amplifier schematic
Parts:
- U1: symbol MCU_Microchip_ATmega:ATmega328P-PU -> PCM-Player-rescue:ATmega328P-PU-MCU_Microchip_ATmega
Changed lines of the file:
@@
 EESchema Schematic File Version 4
-LIBS:PCM Player-cache
-EELAYER 29 0
+EELAYER 30 0
 EELAYER END
 $Descr A4 11693 8268
 encoding utf-8
-Sheet 2 3
+Sheet 2 4
 Title "PCM Player"
 Date "2020-05-07"
@@
 $EndDescr
 $Comp
-L MCU_Microchip_ATmega:ATmega328P-PU U1
+L PCM-Player-rescue:ATmega328P-PU-MCU_Microchip_ATmega U1
 U 1 1 5EB47D68
 P 2850 2750
+AR Path="/5EB47D68" Ref="U1"  Part="1"
+AR Path="/5EB47CA7/5EB47D68" Ref="U1"  Part="1"
 F 0 "U1" H 2206 2796 50  0000 R CNN
 F 1 "ATmega328P-PU" H 2206 2705 50  0000 R CNN
