File: hardware/PCM Player.kicad_pcb (KiCad board)
At the start: 2 copper layers, 0 parts

Commit message: Updated PCB
Parts:
- added C1: 1u, Capacitor_THT:C_Rect_L7.2mm_W4.5mm_P5.00mm_FKS2_FKP2_MKS2_MKP2, F.Cu at (77.5, 52.1)
- added C2: 22p, Capacitor_THT:C_Disc_D3.8mm_W2.6mm_P2.50mm, F.Cu at (52.1, 58.4)
- added C3: 22p, Capacitor_THT:C_Disc_D3.8mm_W2.6mm_P2.50mm, F.Cu at (52.1, 50.8)
- added C4: 4700u, Capacitor_THT:CP_Radial_D16.0mm_P7.50mm, F.Cu at (114.3, 40.6)
- added C5: 100u, Capacitor_THT:CP_Radial_D8.0mm_P3.50mm, F.Cu at (102.9, 40.6)
- added C6: 1u, Capacitor_THT:C_Rect_L7.2mm_W4.5mm_P5.00mm_FKS2_FKP2_MKS2_MKP2, F.Cu at (92.7, 40.6)
- added D1: GBU808, Diode_THT:Diode_Bridge_Vishay_GBU, F.Cu at (114.3, 26.7)
- added F1: 250V 4A, Fuse:Fuseholder_Cylinder-5x20mm_Schurter_0031_8201_Horizontal_Open, F.Cu at (104.1, 61.0)
- added H1: MountingHole, MountingHole:MountingHole_3.2mm_M3, F.Cu at (39.4, 22.9)
- added H2: MountingHole, MountingHole:MountingHole_3.2mm_M3, F.Cu at (39.4, 82.5)
- added H3: MountingHole, MountingHole:MountingHole_3.2mm_M3, F.Cu at (142.2, 22.9)
- added H4: MountingHole, MountingHole:MountingHole_3.2mm_M3, F.Cu at (142.2, 82.5)
- added U1: ATmega328P-PU, Package_DIP:DIP-28_W7.62mm, F.Cu at (63.4, 32.1)
- added U2: LM1085-5.0, Package_TO_SOT_THT:TO-220-3_Vertical, F.Cu at (100.3, 27.9)
- added U3: LP2950-3.3_TO92, Package_TO_SOT_THT:TO-92_Inline, F.Cu at (91.4, 27.9)
- added Y1: 16MHz, Crystal:Crystal_HC49-U_Vertical, F.Cu at (58.4, 55.9)
Other:
- board text added: "CAUTION! Risk of electric shock AC voltage line. Please do not touch this PCB."
- board text added: "MCU"
- board text added: "PSU"
